File: controller_pcb/idk/controller_pcb.kicad_sch (KiCad schematic)
At the start: 22 parts, among them IC1 AMS1117-5.0, J1 A_08-LC-TT, J2 SM03B-GHS-TB_LF__SN_, Q1 SI2301CDS-T1-GE3.

Commit message: MOSFET, regulator, PWR_LED, JST added; half routed; ground plane created
Parts:
- removed J2: SM03B-GHS-TB_LF__SN_, Controller_Footprints:SM03BGHSTBLFSN, symbol Controller_Comp:SM03B-GHS-TB_LF__SN_
- removed LED1: 150080RS75000, Controller_Footprints:LEDC2012X70N, symbol Controller_Comp:150080RS75000
- removed Q1: SI2301CDS-T1-GE3., Controller_Footprints:SOT95P237X112-3N, symbol Controller_Comp:SI2301CDS-T1-GE3.
- removed R6: ERJ-6ENF2200V, Controller_Footprints:ERJ6ENF1000V, symbol Controller_Comp:ERJ-6ENF2200V
- added V1: 1, symbol Simulation_SPICE:VDC
Connections:
- net GND: now also V1.2
- net at C6.1, IC1.3 (VIN): now also V1.1
Other:
- moved on the sheet: C6
