File: controller_pcb/Components/JST (SM04B-GHS-TB)/controller_pcb/controller_pcb.kicad_pcb (KiCad board)
At the start: 2 copper layers, 64.5 x 53.5 mm, 28 parts, among them J1 A_08-LC-TT, J2 SM04B-GHS-TB_LF__SN_, Q1 SI2301CDS-T1-GE3.

Commit message: Silkscreen labels and Baja logo
Parts:
- removed G***: LOGO, Controller_Footprints:BajaLogo2
- renumbered BC to C6, VREG to IC1, PWR to LED1
Routing:
- net Net-(J1-Pad6): track 58.8 -> 52.7 mm
- net Net-(J1-Pad7): track 45.6 -> 39.7 mm
- net Net-(J1-Pad5): track 78.4 -> 76.9 mm, vias 4 -> 2
